Commit message: rename world.launch

File: urdf/slam_project.xacro (robot description, xacro)
@@ -150,5 +150,5 @@
     <joint_properties damping="1.0" friction="1.0"/>
   </joint>
-  <link name='camera'>
+  <link name='camera_link'>
     <inertial>
       <mass value=".1"/>
@@ -160,5 +160,5 @@
       />
     </inertial>
-    <collision name='camera_collision'>
+    <collision name='camera_link_collision'>
       <origin xyz="0 0 0" rpy=" 0 0 0"/>
       <geometry>
@@ -166,5 +166,5 @@
       </geometry>
     </collision>
-    <visual name='camera_visual'>
+    <visual name='camera_link_visual'>
       <origin xyz="0 0 0" rpy=" 0 0 0"/>
       <geometry>
@@ -173,9 +173,15 @@
     </visual>
   </link>
-  <joint type="fixed" name="camera_joint">
+  <joint type="fixed" name="camera_link_joint">
     <origin xyz="0.2 0 0" rpy="0 0 0"/>
-    <child link="camera"/>
-    <parent link="chassis"/>
-  </joint>
+    <child link="camera_link"/>
+    <parent link="chassis"/>
+  </joint>
+  <joint name="camera_joint" type="fixed">
+   <origin xyz="0 0 0" rpy="-1.5707 0 -1.5707"/>
+   <parent link="camera_link"/>
+   <child link="camera_rgbd_frame"/>
+  </joint>
+  <link name="camera_rgbd_frame"/>
   <link name='hokuyo'>
     <inertial>
@@ -197,5 +203,5 @@
       <origin xyz="0 0 0" rpy=" 0 0 0"/>
       <geometry>
-        <mesh filename="package://udacity_bot/meshes/hokuyo.dae"/>
+        <mesh filename="package://slam_project/meshes/hokuyo.dae"/>
       </geometry>
     </visual>
